File: Bitris PCB/BitrisPCB/BitrisATMEGA.brd (EAGLE design)
At the start: 49.2 x 50.8 mm, 27 parts, among them IC1 ATMEGA328-20P, IC2 4511N, X1 Boton, X2 Sonido, X3 Alimentacion, X4 22-23-2021

Commit message: PCB modificado
Parts:
- removed R6: (no value), rcl:M0805
Connections:
- removed net N$34: IC1.1, R6.2, X4.2
- new net N$30: IC1.2, X4.2
- net VCC: no longer R6.1
Routing:
- net VCC: track 122.5 -> 103.3 mm
- net N$34: track 13.0 -> 0.00 mm
- net N$30: track 0.00 -> 8.67 mm
Changed lines of the file:
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@@
 <attribute name="SPICEPREFIX" value="R" x="78.74" y="38.1" size="1.778" layer="27" display="off"/>
-</element>
-<element name="R6" library="rcl" package="M0805" value="" x="39.37" y="46.99" rot="R270">
-<attribute name="SPICEPREFIX" value="R" x="39.37" y="46.99" size="1.778" layer="27" rot="R270" display="off"/>
 </element>
 <element name="R7" library="rcl" package="M0805" value="" x="78.74" y="40.64">
@@
 <contactref element="X3" pad="1"/>
 <contactref element="IC2" pad="16"/>
-<contactref element="R6" pad="1"/>
 <wire x1="67.31" y1="38.1" x2="67.31" y2="39.37" width="1.016" layer="1"/>
 <wire x1="52.07" y1="30.48" x2="54.61" y2="30.48" width="1.016" layer="1"/>
@@
 <wire x1="54.61" y1="50.8" x2="55.88" y2="50.8" width="1.016" layer="1"/>
 <wire x1="55.88" y1="50.8" x2="57.15" y2="49.53" width="1.016" layer="1"/>
-<wire x1="39.37" y1="47.94" x2="39.37" y2="49.53" width="1.016" layer="1"/>
-<wire x1="39.37" y1="49.53" x2="40.64" y2="50.8" width="1.016" layer="1"/>
-<wire x1="40.64" y1="50.8" x2="52.07" y2="50.8" width="1.016" layer="1"/>
-<wire x1="52.07" y1="50.8" x2="54.61" y2="50.8" width="1.016" layer="1"/>
 <wire x1="59.69" y1="27.94" x2="59.69" y2="25.4" width="1.016" layer="1"/>
 <wire x1="55.88" y1="50.8" x2="58.42" y2="50.8" width="1.016" layer="1"/>
@@
 <wire x1="74.93" y1="45.72" x2="73.66" y2="45.72" width="1.016" layer="1"/>
 <wire x1="73.66" y1="45.72" x2="72.39" y2="45.72" width="1.016" layer="1"/>
-<wire x1="52.07" y1="50.8" x2="53.34" y2="52.07" width="1.016" layer="1"/>
 <wire x1="72.39" y1="44.45" x2="73.66" y2="45.72" width="1.016" layer="1"/>
 <wire x1="73.66" y1="45.72" x2="72.39" y2="46.99" width="1.016" layer="1"/>
@@
 <wire x1="39.37" y1="38.1" x2="44.45" y2="38.1" width="1.016" layer="1"/>
 </signal>
-<signal name="N$34">
-<contactref element="IC1" pad="1"/>
-<contactref element="R6" pad="2"/>
-<contactref element="X4" pad="2"/>
-<wire x1="52.07" y1="45.72" x2="44.45" y2="45.72" width="1.016" layer="1"/>
-<wire x1="44.45" y1="45.72" x2="39.37" y2="45.72" width="1.016" layer="1"/>
-<wire x1="39.37" y1="45.72" x2="39.37" y2="46.04" width="1.016" layer="1"/>
-</signal>
 <signal name="N$23">
 <contactref element="IC2" pad="10"/>
@@
 <wire x1="48.26" y1="17.78" x2="52.07" y2="17.78" width="1.016" layer="1"/>
 </signal>
+<signal name="N$30">
+<contactref element="IC1" pad="2"/>
+<contactref element="X4" pad="2"/>
+<wire x1="52.07" y1="43.18" x2="49.53" y2="43.18" width="1.016" layer="1"/>
+<wire x1="49.53" y1="43.18" x2="46.99" y2="45.72" width="1.016" layer="1"/>
+<wire x1="46.99" y1="45.72" x2="44.45" y2="45.72" width="1.016" layer="1"/>
+</signal>
 </signals>

Commit message: PCB 2.0
Parts:
- added R6: (no value), rcl:M0805
- C1: device rcl:C025-025X050 -> rcl:C0805
- C2, C3: value (none) -> 22pf; device rcl:C025-025X050 -> rcl:C0805
- R4: device rcl:M0805 -> rcl:0204/5
- X4: value 22-23-2021 -> Monedas
- moved R4 3.81 mm to (49.5, 48.3)
- moved C1 1.27 mm to (40.6, 39.4)
- moved C2 1.27 mm to (40.6, 26.7)
- moved C3 1.27 mm to (40.6, 21.6)
Connections:
- new net N$34: IC1.1, R6.2
- net VCC: now also R6.1
Routing:
- net VCC: track 103.3 -> 111.1 mm
- net N$4: track 7.94 -> 2.54 mm
- net GND: track 138.6 -> 143.0 mm
- net N$34: track 0.00 -> 3.39 mm
- net N$17: track 17.0 -> 18.8 mm
- net N$33: track 12.7 -> 11.6 mm
- net N$20: track 14.2 -> 13.2 mm
- net N$19: track 13.2 -> 12.2 mm
- added copper zone on layer 1, net N$42
Other:
- board text added: "7°1°"
- board text added: "Campos"
- board text added: "Obregón"
- board text added: "Perez"

Commit message: Limpieza del diseño principal
Parts:
- R1, R10, R11, R12, R2, R3, R4, R5, R7, R8, R9: value (none) -> 220
- R6: value (none) -> 10k
- renumbered JP1 to 7SEG, JP2 to COLUMNA.1, JP3 to COLUMNA.2
Routing:
- net N$41: track 2.86 -> 0.00 mm
- net N$40: track 2.86 -> 0.00 mm
- net N$39: track 2.86 -> 0.00 mm

Commit message: Ajuste SCH
Parts:
- removed COLUMNA.2: (no value), pinhead:1X01
- added JP3: (no value), pinhead:1X01
- added R13, R14: (no value), rcl:M0805
- R1, R10, R11, R12, R2, R3, R4, R5, R7, R8, R9: value 220 -> (none)
- R6: value 10k -> (none)
- X4: value Monedas -> MONEDA; device con-molex:22-23-2021 -> con-molex:22-23-2031
- moved R4 2.54 mm to (49.5, 50.8)
- moved R6 2.54 mm to (49.5, 50.8)
- moved X3 2.54 mm to (58.4, 54.6)
- moved X4 1.27 mm to (44.5, 45.7)
- turned X1 to 90 degrees
- turned X2 to 90 degrees
- renumbered 7SEG to JP1, COLUMNA.1 to JP2
Connections:
- new net N$44: R13.2, X4.3
- net GND: now also X1.2, X2.1; no longer X1.1, X2.2
- net N$30: now also R14.1
- net N$32: now also X2.2; no longer X2.1
- net N$33: now also X1.1; no longer X1.2
- net N$4: now also JP3.1; no longer COLUMNA.2.1
- net VCC: now also R13.1, R14.2
Routing:
- net VCC: track 111.1 -> 144.4 mm
- net N$16: track 4.34 -> 10.5 mm
- net GND: track 143.0 -> 137.9 mm
- net N$44: track 0.00 -> 2.86 mm
- net N$41: track 0.00 -> 2.86 mm
- net N$40: track 0.00 -> 2.86 mm
- net N$39: track 0.00 -> 2.86 mm
- net N$30: track 8.67 -> 11.5 mm
- net N$34: track 3.39 -> 5.93 mm
- net N$17: track 18.8 -> 20.6 mm

Commit message: Actualizado informe
Parts:
- C1: value (none) -> 100nF
- Q1: value (none) -> 16Mhz
- R1, R10, R11, R12, R13, R2, R3, R4, R5, R7, R8, R9: value (none) -> 220
- R14, R6: value (none) -> 10K
- renumbered JP2 to COLUMNAS1, JP3 to COLUMNAS
