File: Bitris PCB/BitrisPCB/BitrisATMEGA.sch (EAGLE design)
At the start: 27 parts, among them IC1 ATMEGA328-20P, IC2 4511N, X1 Boton, X2 Sonido, X3 Alimentacion, X4 22-23-2021

Commit message: PCB modificado
Parts:
- removed R6: (no value), rcl:R-US_M0805
Connections:
- removed net N$34: IC1.PC6(/RESET/PCI14), R6.2, X4-2.S
- new net N$30: IC1.(PCI16/RXD)PD0, X4-2.S
- net VCC: no longer R6.1
Other:
- moved on the sheet: X4-2
Changed lines of the file:
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@@
 <part name="P+5" library="supply1" deviceset="VCC" device=""/>
 <part name="SUPPLY5" library="supply2" deviceset="GND" device=""/>
-<part name="P+6" library="supply1" deviceset="VCC" device=""/>
 <part name="SUPPLY6" library="supply2" deviceset="GND" device=""/>
-<part name="R6" library="rcl" deviceset="R-US_" device="M0805"/>
 <part name="R5" library="rcl" deviceset="R-US_" device="M0805"/>
 <part name="R7" library="rcl" deviceset="R-US_" device="M0805"/>
@@
 <attribute name="VALUE" x="135.255" y="24.765" size="1.778" layer="96"/>
 </instance>
-<instance part="P+6" gate="VCC" x="2.54" y="101.6" smashed="yes">
-<attribute name="VALUE" x="0" y="99.06" size="1.778" layer="96" rot="R90"/>
-</instance>
 <instance part="SUPPLY6" gate="GND" x="15.24" y="99.06" smashed="yes">
 <attribute name="VALUE" x="13.335" y="95.885" size="1.778" layer="96"/>
-</instance>
-<instance part="R6" gate="G$1" x="7.62" y="96.52" smashed="yes">
-<attribute name="NAME" x="3.81" y="98.0186" size="1.778" layer="95"/>
-<attribute name="VALUE" x="3.81" y="93.218" size="1.778" layer="96"/>
 </instance>
 <instance part="R5" gate="G$1" x="134.62" y="60.96" smashed="yes">
@@
 </instance>
 <instance part="X4" gate="-1" x="17.78" y="109.22" rot="R90"/>
-<instance part="X4" gate="-2" x="20.32" y="109.22" rot="R90"/>
+<instance part="X4" gate="-2" x="73.66" y="73.66" rot="R90"/>
 <instance part="JP2" gate="A" x="142.24" y="93.98"/>
 <instance part="JP3" gate="G$1" x="142.24" y="83.82"/>
@@
 <pinref part="IC2" gate="P" pin="VDD"/>
 <pinref part="P+5" gate="VCC" pin="VCC"/>
-</segment>
-<segment>
-<pinref part="P+6" gate="VCC" pin="VCC"/>
-<pinref part="R6" gate="G$1" pin="1"/>
-<wire x1="2.54" y1="99.06" x2="2.54" y2="96.52" width="0.1524" layer="91"/>
 </segment>
 </net>
@@
 </segment>
 </net>
-<net name="N$34" class="0">
-<segment>
-<pinref part="IC1" gate="G$1" pin="PC6(/RESET/PCI14)"/>
-<wire x1="12.7" y1="96.52" x2="17.78" y2="96.52" width="0.1524" layer="91"/>
-<wire x1="20.32" y1="96.52" x2="17.78" y2="96.52" width="0.1524" layer="91"/>
-<pinref part="R6" gate="G$1" pin="2"/>
-<pinref part="X4" gate="-2" pin="S"/>
-<wire x1="20.32" y1="106.68" x2="20.32" y2="96.52" width="0.1524" layer="91"/>
-</segment>
-</net>
 <net name="N$23" class="0">
 <segment>
@@
 </segment>
 </net>
+<net name="N$30" class="0">
+<segment>
+<pinref part="IC1" gate="G$1" pin="(PCI16/RXD)PD0"/>
+<pinref part="X4" gate="-2" pin="S"/>
+</segment>
+</net>

Commit message: PCB 2.0
Parts:
- added R6: (no value), rcl:R-US_M0805
- C1: device rcl:C-US025-025X050 -> rcl:C-USC0805
- C2, C3: value (none) -> 22pf; device rcl:C-US025-025X050 -> rcl:C-USC0805
- R4: device rcl:R-US_M0805 -> rcl:R-US_0204/5
- X4: value 22-23-2021 -> Monedas
Connections:
- new net N$34: IC1.PC6(/RESET/PCI14), R6.2
- net VCC: now also R6.1
Changed lines of the file:
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@@
 <part name="R2" library="rcl" deviceset="R-US_" device="M0805"/>
 <part name="R3" library="rcl" deviceset="R-US_" device="M0805"/>
-<part name="R4" library="rcl" deviceset="R-US_" device="M0805"/>
+<part name="R4" library="rcl" deviceset="R-US_" device="0204/5"/>
 <part name="FILAS" library="pinhead" deviceset="PINHD-1X6" device=""/>
 <part name="IC2" library="45xx" deviceset="4511" device="N"/>
@@
 <part name="MULTI" library="pinhead" deviceset="PINHD-1X2" device=""/>
 <part name="SUPPLY4" library="supply2" deviceset="GND" device=""/>
-<part name="C1" library="rcl" deviceset="C-US" device="025-025X050"/>
-<part name="C2" library="rcl" deviceset="C-US" device="025-025X050"/>
-<part name="C3" library="rcl" deviceset="C-US" device="025-025X050"/>
+<part name="C1" library="rcl" deviceset="C-US" device="C0805"/>
+<part name="C2" library="rcl" deviceset="C-US" device="C0805" value="22pf"/>
+<part name="C3" library="rcl" deviceset="C-US" device="C0805" value="22pf"/>
 <part name="P+4" library="supply1" deviceset="VCC" device=""/>
 <part name="SUPPLY2" library="supply2" deviceset="GND" device=""/>
@@
 <part name="R11" library="rcl" deviceset="R-US_" device="M0805"/>
 <part name="R12" library="rcl" deviceset="R-US_" device="M0805"/>
-<part name="X4" library="con-molex" deviceset="22-23-2021" device=""/>
+<part name="X4" library="con-molex" deviceset="22-23-2021" device="" value="Monedas"/>
 <part name="JP2" library="pinhead" deviceset="PINHD-1X3" device=""/>
 <part name="JP3" library="pinhead" deviceset="PINHD-1X1" device=""/>
+<part name="R6" library="rcl" deviceset="R-US_" device="M0805"/>
 </parts>
 <sheets>
@@
 <instance part="JP2" gate="A" x="142.24" y="93.98"/>
 <instance part="JP3" gate="G$1" x="142.24" y="83.82"/>
+<instance part="R6" gate="G$1" x="5.08" y="99.06"/>
 </instances>
 <busses>
@@
 <wire x1="-17.78" y1="104.14" x2="-12.7" y2="104.14" width="0.1524" layer="91"/>
 <wire x1="-12.7" y1="104.14" x2="-12.7" y2="106.68" width="0.1524" layer="91"/>
+<pinref part="R6" gate="G$1" pin="1"/>
+<wire x1="0" y1="99.06" x2="0" y2="104.14" width="0.1524" layer="91"/>
+<wire x1="-12.7" y1="104.14" x2="0" y2="104.14" width="0.1524" layer="91"/>
+<junction x="-12.7" y="104.14"/>
 </segment>
 <segment>
@@
 </segment>
 </net>
+<net name="N$34" class="0">
+<segment>
+<pinref part="IC1" gate="G$1" pin="PC6(/RESET/PCI14)"/>
+<pinref part="R6" gate="G$1" pin="2"/>
+<wire x1="17.78" y1="96.52" x2="10.16" y2="96.52" width="0.1524" layer="91"/>
+<wire x1="10.16" y1="96.52" x2="10.16" y2="99.06" width="0.1524" layer="91"/>
+</segment>
+</net>

Commit message: Limpieza del diseño principal
Parts:
- removed JP1: (no value), pinhead:PINHD-1X7
- removed JP2: (no value), pinhead:PINHD-1X3
- removed JP3: (no value), pinhead:PINHD-1X1
- added 7SEG: (no value), pinhead:PINHD-1X7
- added COLUMNA.1: (no value), pinhead:PINHD-1X3
- added COLUMNA.2: (no value), pinhead:PINHD-1X1
- R1, R10, R11, R12, R2, R3, R4, R5, R7, R8, R9: value (none) -> 220
- R6: value (none) -> 10k
Connections:
- net N$1: now also COLUMNA.1.1; no longer JP2.1
- net N$2: now also COLUMNA.1.2; no longer JP2.2
- net N$3: now also COLUMNA.1.3; no longer JP2.3
- net N$35: now also 7SEG.1; no longer JP1.1
- net N$36: now also 7SEG.2; no longer JP1.2
- net N$37: now also 7SEG.3; no longer JP1.3
- net N$38: now also 7SEG.4; no longer JP1.4
- net N$39: now also 7SEG.5; no longer JP1.5
- net N$4: now also COLUMNA.2.1; no longer JP3.1
- net N$40: now also 7SEG.6; no longer JP1.6
- net N$41: now also 7SEG.7; no longer JP1.7
Other:
- moved on the sheet: R1, R10, R11, R12, R2, R3, R4, R5, R6, R7, R8, R9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

Commit message: Ajuste SCH
Parts:
- removed 7SEG: (no value), pinhead:PINHD-1X7
- removed COLUMNA.1: (no value), pinhead:PINHD-1X3
- removed COLUMNA.2: (no value), pinhead:PINHD-1X1
- added JP1: (no value), pinhead:PINHD-1X7
- added JP2: (no value), pinhead:PINHD-1X3
- added JP3: (no value), pinhead:PINHD-1X1
- added R13, R14: (no value), rcl:R-US_M0805
- R1, R10, R11, R12, R2, R3, R4, R5, R7, R8, R9: value 220 -> (none)
- R6: value 10k -> (none)
- X4: value Monedas -> MONEDA; device con-molex:22-23-2021 -> con-molex:22-23-2031
Connections:
- new net N$44: R13.2, X4-3.S
- net GND: now also X1-2.S, X2-1.S; no longer X1-1.S, X2-2.S
- net N$1: now also JP2.1; no longer COLUMNA.1.1
- net N$2: now also JP2.2; no longer COLUMNA.1.2
- net N$3: now also JP2.3; no longer COLUMNA.1.3
- net N$30: now also R14.1
- net N$32: now also X2-2.S; no longer X2-1.S
- net N$33: now also X1-1.S; no longer X1-2.S
- net N$35: now also JP1.1; no longer 7SEG.1
- net N$36: now also JP1.2; no longer 7SEG.2
- net N$37: now also JP1.3; no longer 7SEG.3
- net N$38: now also JP1.4; no longer 7SEG.4
- net N$39: now also JP1.5; no longer 7SEG.5
- net N$4: now also JP3.1; no longer COLUMNA.2.1
- net N$40: now also JP1.6; no longer 7SEG.6
- net N$41: now also JP1.7; no longer 7SEG.7
- net VCC: now also R13.1, R14.2
Other:
- moved on the sheet: R1, R2, R3, R4, R6, R8, X1-1, X1-2, X2-1, X2-2, X3-1, X3-2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

Commit message: Actualizado informe
Parts:
- removed JP2: (no value), pinhead:PINHD-1X3
- removed JP3: (no value), pinhead:PINHD-1X1
- added COLUMNAS: (no value), pinhead:PINHD-1X1
- added COLUMNAS1: (no value), pinhead:PINHD-1X3
- C1: value (none) -> 100nF
- Q1: value (none) -> 16Mhz
- R1, R10, R11, R12, R13, R2, R3, R4, R5, R7, R8, R9: value (none) -> 220
- R14, R6: value (none) -> 10K
Connections:
- net N$1: now also COLUMNAS1.1; no longer JP2.1
- net N$2: now also COLUMNAS1.2; no longer JP2.2
- net N$3: now also COLUMNAS1.3; no longer JP2.3
- net N$4: now also COLUMNAS.1; no longer JP3.1
Other:
- moved on the sheet: C1, C2, C3, FILAS, IC1, IC2, IC2P, JP1, MULTI, Q1, R1, R10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
